File: Bridge/Bridge.kicad_pcb (KiCad board)
At the start: 2 copper layers, 95 x 72 mm, 31 parts, among them J1 Conn_01x01_Pin, J2 Conn_01x01_Pin, J3 Conn_01x01_Pin, J4 Conn_01x02_Pin, J5 Barrel_Jack, Q1 BUZ11, Q2 BUZ11, U1 74132, U2 TLP250, U3 TLP250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

Commit message: edit silkscreen
Connections:
- HS1 pad 1: GND -> unconnected-(HS1-Pad1)
- HS1 pad 2: GND -> unconnected-(HS1-Pad2)
- HS2 pad 1: GND -> unconnected-(HS2-Pad1)
- HS2 pad 2: GND -> unconnected-(HS2-Pad2)
Routing:
- net GND: track 97.0 -> 95.9 mm
Other:
- board text added: "GND"
- board text added: "Phase :"
- board text added: "Signal"
- board text added: "https://github.com/53175ddd/3P-VVVF"
Changed lines of the file:
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@@
   (net 24 "unconnected-(U3-NC-Pad1)")
   (net 25 "unconnected-(U3-NC-Pad4)")
+  (net 26 "unconnected-(HS1-Pad1)")
+  (net 27 "unconnected-(HS1-Pad2)")
+  (net 28 "unconnected-(HS2-Pad1)")
+  (net 29 "unconnected-(HS2-Pad2)")
   (footprint "Resistor_THT:R_Axial_DIN0204_L3.6mm_D1.6mm_P7.62mm_Horizontal" (layer "F.Cu")
     (at 109.22 107.95 90)
@@
       (stroke (width 0.1) (type default)) (layer "F.SilkS"))
     (pad "1" thru_hole circle (at -5 0 270) (size 3 3) (drill 1.6) (layers "*.Cu" "*.Mask")
-      (net 5 "GND") (pintype "passive"))
+      (net 26 "unconnected-(HS1-Pad1)") (pintype "passive+no_connect"))
     (pad "2" thru_hole circle (at 5 0 270) (size 3 3) (drill 1.6) (layers "*.Cu" "*.Mask")
-      (net 5 "GND") (pintype "passive"))
+      (net 27 "unconnected-(HS1-Pad2)") (pintype "passive+no_connect"))
   )
   (footprint "Capacitor_THT:C_Disc_D6.0mm_W2.5mm_P5.00mm" (layer "F.Cu")
@@
       (stroke (width 0.1) (type default)) (layer "F.SilkS"))
     (pad "1" thru_hole circle (at -5 0 270) (size 3 3) (drill 1.6) (layers "*.Cu" "*.Mask")
-      (net 5 "GND") (pintype "passive"))
+      (net 28 "unconnected-(HS2-Pad1)") (pintype "passive+no_connect"))
     (pad "2" thru_hole circle (at 5 0 270) (size 3 3) (drill 1.6) (layers "*.Cu" "*.Mask")
-      (net 5 "GND") (pintype "passive"))
+      (net 29 "unconnected-(HS2-Pad2)") (pintype "passive+no_connect"))
   )
   (footprint "Resistor_THT:R_Axial_DIN0204_L3.6mm_D1.6mm_P7.62mm_Horizontal" (layer "F.Cu")
@@
   (gr_circle (center 107.9 68.6) (end 109.5 68.6)
     (stroke (width 0.1) (type default)) (fill none) (layer "Edge.Cuts"))
+  (gr_text "https://github.com/53175ddd/3P-VVVF" (at 193.04 133.35) (layer "B.SilkS")
+    (effects (font (size 2 2) (thickness 0.2)) (justify left top mirror))
+  )
+  (gr_text "GND" (at 109.855 95.885) (layer "F.SilkS")
+    (effects (font (size 1 1) (thickness 0.15)) (justify left bottom))
+  )
+  (gr_text "Signal" (at 109.855 93.345) (layer "F.SilkS")
+    (effects (font (size 1 1) (thickness 0.15)) (justify left bottom))
+  )
   (gr_text "Half Bridge Inverter v1\nPCB by MOS@53175DDD" (at 112.395 135.89) (layer "F.SilkS")
     (effects (font (size 2 2) (thickness 0.2)) (justify left bottom))
+  )
+  (gr_text "Phase : " (at 154.94 134.62) (layer "F.SilkS")
+    (effects (font (size 3 3) (thickness 0.3) bold) (justify left bottom))
   )
   (segment (start 177.546 84.836) (end 177.4825 84.7725) (width 3) (layer "F.Cu") (net 1))
@@
   (segment (start 195.66 125.476) (end 185.506 125.476) (width 3) (layer "F.Cu") (net 5))
   (segment (start 195.66 118.37) (end 183.89 118.37) (width 3) (layer "F.Cu") (net 5))
-  (segment (start 134.63 118.12) (end 132.08 115.57) (width 1) (layer "F.Cu") (net 5))
   (segment (start 185.506 125.476) (end 185.5 125.482) (width 3) (layer "F.Cu") (net 5))
   (segment (start 157.48 117.21) (end 154.04 117.21) (width 1) (layer "F.Cu") (net 5))
   (segment (start 152.4 115.57) (end 146.05 115.57) (width 1) (layer "F.Cu") (net 5))
   (segment (start 183.902 125.482) (end 185.5 125.482) (width 3) (layer "F.Cu") (net 5))
+  (segment (start 132.08 118.11) (end 131.445 118.11) (width 1) (layer "F.Cu") (net 5))
   (segment (start 154.04 117.21) (end 152.4 115.57) (width 1) (layer "F.Cu") (net 5))
-  (segment (start 132.08 115.57) (end 131.445 115.57) (width 1) (layer "F.Cu") (net 5))
   (segment (start 138.38 118.12) (end 139.7 116.8) (width 1) (layer "F.Cu") (net 5))
   (segment (start 154.04 117.21) (end 147.69 117.21) (width 1) (layer "F.Cu") (net 5))
   (segment (start 183.89 118.37) (end 180.34 121.92) (width 3) (layer "F.Cu") (net 5))
   (segment (start 162.19 121.92) (end 157.48 117.21) (width 3) (layer "F.Cu") (net 5))
-  (segment (start 132.08 115.57) (end 132.07 115.58) (width 1) (layer "F.Cu") (net 5))
-  (segment (start 137.17 118.12) (end 134.63 118.12) (width 1) (layer "F.Cu") (net 5))
+  (segment (start 132.09 118.12) (end 132.08 118.11) (width 1) (layer "F.Cu") (net 5))
   (segment (start 180.34 121.92) (end 162.19 121.92) (width 3) (layer "F.Cu") (net 5))
   (segment (start 146.05 115.57) (end 144.78 114.3) (width 1) (layer "F.Cu") (net 5))
+  (segment (start 137.17 118.12) (end 132.09 118.12) (width 1) (layer "F.Cu") (net 5))
   (segment (start 147.69 117.21) (end 146.05 115.57) (width 1) (layer "F.Cu") (net 5))
   (segment (start 137.17 118.12) (end 138.38 118.12) (width 1) (layer "F.Cu") (net 5))
@@
       )
     )
+  )
+  (zone (net 0) (net_name "") (layer "F.SilkS") (hatch edge 0.5)
+    (connect_pads (clearance 0.5))
+    (min_thickness 0.25) (filled_areas_thickness no)
+    (fill yes (thermal_gap 0.5) (thermal_bridge_width 0.5))
+    (polygon
+      (pts
+        (xy 172.72 136.525)
+        (xy 179.705 136.525)
+        (xy 179.705 130.175)
+        (xy 172.72 130.175)
+      )
+    )

Commit message: PCB を v2 に update
Parts:
- moved U4 1.31 mm to (120.0, 87.7)
- moved C8 1.31 mm to (116.2, 87.7)
- moved C9 1.27 mm to (120.0, 97.8)
Routing:
- net +5V: track 10.4 -> 9.11 mm
- net +12V: track 65.1 -> 66.4 mm
- net Net-(R4-Pad1): track 26.7 -> 26.0 mm
- net Net-(R3-Pad1): track 26.7 -> 26.0 mm
- net GND: vias 202 -> 219
Other:
- board text added: "Half Bridge Inverter v2 PCB by MOS@53175DDD"
- board text removed: "Half Bridge Inverter v1 PCB by MOS@53175DDD"
